File: engineers thumb.kicad_pcb (KiCad board)
At the start: 2 copper layers, 86.4 x 63.5 mm, 55 parts, among them J1 INPUT, J2 GND, J3 9V, J4 GND, J5 LED+, J6 Out, Q1 Q_PMOS_GSD, Q2 BC327, SW1 TREBLE_BOOST, U1 TL072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

Commit message: Starting to do changes
Parts:
- removed J5: LED+, Connector_PinSocket_2.54mm:PinSocket_1x01_P2.54mm_Vertical
- removed R21: R_LED, 2.Breadboard components:R_Axial_Horizontal
- J1: value INPUT -> Conn_01x01
- J2, J4: value GND -> Conn_01x01
- J3: value 9V -> Conn_01x01
- J6: value Out -> Conn_01x01
- RV1: value TH -> 1Meg_lin
- RV2: value RATIO -> 1Meg_log
- RV3: value REL -> 1Meg_lin
- RV4: value ATT -> 100k_log
- RV5: value VOLUME -> 10k_log
- SW1: value TREBLE_BOOST -> SPST
Routing:
- net Net-(J5-Pad1): track 7.62 -> 0.00 mm, vias 1 -> 0
- net +9V: track 191.6 -> 186.5 mm, vias 6 -> 5
Other:
- board text removed: "LED+"
Changed lines of the file:
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@@
   (general
     (thickness 1.6)
-    (drawings 10)
-    (tracks 283)
+    (drawings 9)
+    (tracks 278)
     (zones 0)
-    (modules 55)
-    (nets 34)
+    (modules 53)
+    (nets 33)
   )
   (page A4)
@@
   (net 31 "Net-(D2-Pad2)")
   (net 32 "Net-(J3-Pad1)")
-  (net 33 "Net-(J5-Pad1)")
   (net_class Default "This is the default net class."
     (clearance 0.508)
@@
     (add_net "Net-(J1-Pad1)")
     (add_net "Net-(J3-Pad1)")
-    (add_net "Net-(J5-Pad1)")
     (add_net "Net-(Q2-Pad1)")
     (add_net "Net-(Q2-Pad2)")
@@
     (add_net "Net-(RV1-Pad2)")
     (add_net "Net-(RV5-Pad2)")
+    (add_net "Net-(U3-Pad15)")
+    (add_net "Net-(U3-Pad2)")
+    (add_net "Net-(U3-Pad9)")
   )
   (module "2.Breadboard components:C_Box_P5.08mm" (layer F.Cu)
@@
       (effects (font (size 1 1) (thickness 0.15)))
     )
-    (fp_text value TH (at 0 5.08) (layer F.Fab)
+    (fp_text value 1Meg_lin (at 0 5.08) (layer F.Fab)
       (effects (font (size 1 1) (thickness 0.15)))
     )
@@
       (effects (font (size 1 1) (thickness 0.15)))
     )
-    (fp_text value TREBLE_BOOST (at 2.54 -2.54 90) (layer F.Fab)
+    (fp_text value SPST (at 2.54 -2.54 90) (layer F.Fab)
       (effects (font (size 1 1) (thickness 0.15)))
     )
@@
       (effects (font (size 1 1) (thickness 0.15)))
     )
-    (fp_text value VOLUME (at 0 5.08) (layer F.Fab)
+    (fp_text value 10k_log (at 0 5.08) (layer F.Fab)
       (effects (font (size 1 1) (thickness 0.15)))
     )
@@
       (effects (font (size 1 1) (thickness 0.15)))
     )
-    (fp_text value ATT (at 0 5.08) (layer F.Fab)
+    (fp_text value 100k_log (at 0 5.08) (layer F.Fab)
       (effects (font (size 1 1) (thickness 0.15)))
     )
@@
       (effects (font (size 1 1) (thickness 0.15)))
     )
-    (fp_text value REL (at 0 5.08) (layer F.Fab)
+    (fp_text value 1Meg_lin (at 0 5.08) (layer F.Fab)
       (effects (font (size 1 1) (thickness 0.15)))
     )
@@
       (effects (font (size 1 1) (thickness 0.15)))
     )
-    (fp_text value RATIO (at 0 5.08) (layer F.Fab)
+    (fp_text value 1Meg_log (at 0 5.08) (layer F.Fab)
       (effects (font (size 1 1) (thickness 0.15)))
     )
@@
   )
   (module "2.Breadboard components:R_Axial_Horizontal" (layer F.Cu)
-    (at 129.54 121.92 90)
-    (descr "Resistor, Axial_DIN0204 series, Axial, Horizontal, pin pitch=7.62mm, 0.167W, length*diameter=3.6*1.6mm^2, http://cdn-reichelt.de/documents/datenblatt/B400/1_4W%23YAG.pdf")
-    (tags "Resistor Axial_DIN0204 series Axial Horizontal pin pitch 7.62mm 0.167W length 3.6mm diameter 1.6mm")
-    (fp_text reference R21 (at -1.905 0 180) (layer F.SilkS)
-      (effects (font (size 1 1) (thickness 0.15)))
-    )
-    (fp_text value R_LED (at 3.81 1.92 90) (layer F.Fab)
-      (effects (font (size 1 1) (thickness 0.15)))
-    )
-    (fp_text user %R (at 3.81 0 90) (layer F.Fab)
-      (effects (font (size 0.72 0.72) (thickness 0.108)))
-    )
-    (fp_line (start 8.3185 -1.0795) (end -0.6985 -1.0795) (layer F.CrtYd) (width 0.05))
-    (fp_line (start 8.3135 1.0795) (end 8.3185 -1.0795) (layer F.CrtYd) (width 0.05))
-    (fp_line (start -0.6985 1.0795) (end 8.3135 1.0795) (layer F.CrtYd) (width 0.05))
-    (fp_line (start -0.6985 -1.0795) (end -0.6985 1.0795) (layer F.CrtYd) (width 0.05))
-    (fp_line (start 6.858 0) (end 6.7945 0) (layer F.SilkS) (width 0.12))
-    (fp_line (start 0.762 0) (end 0.8255 0) (layer F.SilkS) (width 0.12))
-    (fp_line (start 6.7945 -1.016) (end 0.8255 -1.016) (layer F.SilkS) (width 0.12))
-    (fp_line (start 6.7945 1.016) (end 6.7945 -1.016) (layer F.SilkS) (width 0.12))
-    (fp_line (start 0.8255 1.016) (end 6.7945 1.016) (layer F.SilkS) (width 0.12))
-    (fp_line (start 0.8255 -1.016) (end 0.8255 1.016) (layer F.SilkS) (width 0.12))
-    (fp_line (start 7.62 0) (end 6.6675 0) (layer F.Fab) (width 0.1))
-    (fp_line (start 0 0) (end 0.889 0) (layer F.Fab) (width 0.1))
-    (fp_line (start 6.6675 -0.889) (end 0.9525 -0.889) (layer F.Fab) (width 0.1))
-    (fp_line (start 6.6675 0.889) (end 6.6675 -0.889) (layer F.Fab) (width 0.1))
-    (fp_line (start 0.9525 0.889) (end 6.6675 0.889) (layer F.Fab) (width 0.1))
-    (fp_line (start 0.9525 -0.889) (end 0.9525 0.889) (layer F.Fab) (width 0.1))
-    (pad 2 smd oval (at 7.62 0 90) (size 1.4 1.4) (layers F.Cu)
-      (net 2 +9V))
-    (pad 1 smd circle (at 0 0 90) (size 1.4 1.4) (layers F.Cu)
-      (net 33 "Net-(J5-Pad1)"))
-    (model ${KISYS3DMOD}/Resistor_THT.3dshapes/R_Axial_DIN0204_L3.6mm_D1.6mm_P7.62mm_Horizontal.wrl
-      (at (xyz 0 0 0))
-      (scale (xyz 1 1 1))
-      (rotate (xyz 0 0 0))
-    )
-  )
-  (module "2.Breadboard components:R_Axial_Horizontal" (layer F.Cu)
     (at 76.2 127)
     (descr "Resistor, Axial_DIN0204 series, Axial, Horizontal, pin pitch=7.62mm, 0.167W, length*diameter=3.6*1.6mm^2, http://cdn-reichelt.de/documents/datenblatt/B400/1_4W%23YAG.pdf")
@@
       (effects (font (size 1 1) (thickness 0.15)))
     )
-    (fp_text value Out (at 0 2.77) (layer F.Fab)
+    (fp_text value Conn_01x01 (at 0 2.77) (layer F.Fab)
       (effects (font (size 1 1) (thickness 0.15)))
     )
@@
   )
   (module Connector_PinSocket_2.54mm:PinSocket_1x01_P2.54mm_Vertical (layer F.Cu)
-    (at 129.54 129.54)
-    (descr "Through hole straight socket strip, 1x01, 2.54mm pitch, single row (from Kicad 4.0.7), script generated")
-    (tags "Through hole socket strip THT 1x01 2.54mm single row")
-    (fp_text reference J5 (at -2.54 0) (layer F.SilkS)
-      (effects (font (size 1 1) (thickness 0.15)))
-    )
-    (fp_text value LED+ (at 0 2.77) (layer F.Fab)
-      (effects (font (size 1 1) (thickness 0.15)))
-    )
-    (fp_text user %R (at 0 0) (layer F.Fab)
-      (effects (font (size 1 1) (thickness 0.15)))
-    )
-    (fp_line (start -1.8 1.75) (end -1.8 -1.8) (layer F.CrtYd) (width 0.05))
-    (fp_line (start 1.75 1.75) (end -1.8 1.75) (layer F.CrtYd) (width 0.05))
-    (fp_line (start 1.75 -1.8) (end 1.75 1.75) (layer F.CrtYd) (width 0.05))
-    (fp_line (start -1.8 -1.8) (end 1.75 -1.8) (layer F.CrtYd) (width 0.05))
-    (fp_line (start 0 -1.33) (end 1.33 -1.33) (layer F.SilkS) (width 0.12))
-    (fp_line (start 1.33 -1.33) (end 1.33 0) (layer F.SilkS) (width 0.12))
-    (fp_line (start 1.33 1.21) (end 1.33 1.33) (layer F.SilkS) (width 0.12))
-    (fp_line (start -1.33 1.21) (end -1.33 1.33) (layer F.SilkS) (width 0.12))
-    (fp_line (start -1.33 1.33) (end 1.33 1.33) (layer F.SilkS) (width 0.12))
-    (fp_line (start -1.27 1.27) (end -1.27 -1.27) (layer F.Fab) (width 0.1))
-    (fp_line (start 1.27 1.27) (end -1.27 1.27) (layer F.Fab) (width 0.1))
-    (fp_line (start 1.27 -0.635) (end 1.27 1.27) (layer F.Fab) (width 0.1))
-    (fp_line (start 0.635 -1.27) (end 1.27 -0.635) (layer F.Fab) (width 0.1))
-    (fp_line (start -1.27 -1.27) (end 0.635 -1.27) (layer F.Fab) (width 0.1))
-    (pad 1 thru_hole rect (at 0 0) (size 1.7 1.7) (drill 1) (layers *.Cu *.Mask)
-      (net 33 "Net-(J5-Pad1)"))
-    (model ${KISYS3DMOD}/Connector_PinSocket_2.54mm.3dshapes/PinSocket_1x01_P2.54mm_Vertical.wrl
-      (at (xyz 0 0 0))
-      (scale (xyz 1 1 1))
-      (rotate (xyz 0 0 0))
-    )
-  )
-  (module Connector_PinSocket_2.54mm:PinSocket_1x01_P2.54mm_Vertical (layer F.Cu)
     (at 58.42 73.66)
     (descr "Through hole straight socket strip, 1x01, 2.54mm pitch, single row (from Kicad 4.0.7), script generated")
@@
       (effects (font (size 1 1) (thickness 0.15)))
     )
-    (fp_text value GND (at 0 2.77) (layer F.Fab)
+    (fp_text value Conn_01x01 (at 0 2.77) (layer F.Fab)
       (effects (font (size 1 1) (thickness 0.15)))
     )
@@
       (effects (font (size 1 1) (thickness 0.15)))
     )
-    (fp_text value 9V (at 0 2.77) (layer F.Fab)
+    (fp_text value Conn_01x01 (at 0 2.77) (layer F.Fab)
       (effects (font (size 1 1) (thickness 0.15)))
     )
@@
       (effects (font (size 1 1) (thickness 0.15)))
     )
-    (fp_text value GND (at 0 2.77) (layer F.Fab)
+    (fp_text value Conn_01x01 (at 0 2.77) (layer F.Fab)
       (effects (font (size 1 1) (thickness 0.15)))
     )
@@
       (effects (font (size 1 1) (thickness 0.15)))
     )
-    (fp_text value INPUT (at 0 2.77) (layer F.Fab)
+    (fp_text value Conn_01x01 (at 0 2.77) (layer F.Fab)
       (effects (font (size 1 1) (thickness 0.15)))
     )
@@
     )
   )
-  (gr_text LED+ (at 129.54 127) (layer F.SilkS)
-    (effects (font (size 1 1) (thickness 0.15)))
-  )
   (gr_text OUT (at 86.36 127) (layer F.SilkS)
     (effects (font (size 1 1) (thickness 0.15)))
@@
   (segment (start 99.06 99.06) (end 99.06 96.52) (width 0.635) (layer B.Cu) (net 2))
   (segment (start 127 109.22) (end 129.54 109.22) (width 0.635) (layer B.Cu) (net 2))
-  (via (at 129.54 109.22) (size 1.2) (drill 0.8) (layers F.Cu B.Cu) (net 2))
   (segment (start 68.58 86.36) (end 71.12 86.36) (width 0.635) (layer B.Cu) (net 2))
   (segment (start 71.12 86.36) (end 71.12 99.06) (width 0.635) (layer B.Cu) (net 2))
@@
   (via (at 93.98 81.28) (size 1.2) (drill 0.8) (layers F.Cu B.Cu) (net 2))
   (via (at 93.98 76.2) (size 1.2) (drill 0.8) (layers F.Cu B.Cu) (net 2))
-  (segment (start 129.54 114.3) (end 129.54 109.22) (width 0.635) (layer F.Cu) (net 2))
   (segment (start 71.12 86.36) (end 71.12 81.28) (width 0.635) (layer B.Cu) (net 2))
   (segment (start 71.12 81.28) (end 88.9 81.28) (width 0.635) (layer B.Cu) (net 2))
@@
   (segment (start 64.45 74.61) (end 63.5 73.66) (width 0.635) (layer B.Cu) (net 32))
   (segment (start 66.88 74.61) (end 64.45 74.61) (width 0.635) (layer B.Cu) (net 32))
-  (via (at 129.54 127) (size 1.2) (drill 0.8) (layers F.Cu B.Cu) (net 33))
-  (segment (start 129.54 121.92) (end 129.54 127) (width 0.635) (layer F.Cu) (net 33))
-  (segment (start 129.54 127) (end 129.54 129.54) (width 0.635) (layer B.Cu) (net 33))
 )

Commit message: WIP
Parts:
- moved J2 130.6 mm to (177.8, 50.8), turned to 90 degrees
- moved J4 128.8 mm to (177.8, 121.9), turned to 90 degrees
- moved J3 117.7 mm to (177.8, 45.7), turned to 90 degrees
- moved RV2 113.4 mm to (177.8, 91.4), turned to 90 degrees
- moved J1 112.5 mm to (177.8, 116.8), turned to 90 degrees
- moved RV1 110.3 mm to (177.8, 76.2), turned to 90 degrees
- moved R17 106.1 mm to (33.3, 148.3), turned to 0 degrees
- moved R10 104.3 mm to (167.6, 61.0), turned to 180 degrees
- moved RV4 103.6 mm to (177.8, 61.0), turned to 90 degrees
- moved Q1 102.5 mm to (167.6, 48.3), turned to 0 degrees
- moved D2 94.0 mm to (162.6, 45.7), turned to 270 degrees
- moved C3 91.6 mm to (160.0, 81.3), turned to 90 degrees
- moved J6 91.5 mm to (177.8, 127.0), turned to 90 degrees
- moved U1 88.9 mm to (154.9, 104.1), turned to 270 degrees
- moved R3 88.2 mm to (162.6, 53.3), turned to 90 degrees
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Routing:
- net GND: track 317.6 -> 0.00 mm, vias 13 -> 0
- net +9V: track 186.5 -> 0.00 mm, vias 5 -> 0
- net Net-(C5-Pad2): track 106.7 -> 0.00 mm, vias 2 -> 0
- net Net-(C5-Pad1): track 86.4 -> 0.00 mm, vias 2 -> 0
- net +4V5: track 83.8 -> 0.00 mm, vias 4 -> 0
- net Net-(R5-Pad2): track 61.0 -> 0.00 mm, vias 1 -> 0
- net Net-(C8-Pad1): track 58.4 -> 0.00 mm, vias 2 -> 0
- net Net-(C11-Pad2): track 35.6 -> 0.00 mm, vias 4 -> 0
- net Net-(RV5-Pad2): track 35.6 -> 0.00 mm, vias 2 -> 0
- net Net-(Q2-Pad3): track 33.0 -> 0.00 mm, vias 2 -> 0
- net Net-(C2-Pad1): track 27.9 -> 0.00 mm
- net Net-(R6-Pad2): track 22.9 -> 0.00 mm, vias 1 -> 0
- net Net-(RV1-Pad2): track 22.9 -> 0.00 mm
- net Net-(R14-Pad1): track 22.9 -> 0.00 mm, vias 1 -> 0
- net Net-(C7-Pad1): track 22.9 -> 0.00 mm, vias 3 -> 0
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Other:
- board outline removed
- board text removed: "+9V"
- board text removed: "GND"
- board text removed: "IN"
- board text removed: "OUT"

Commit message: Almost done
Parts:
- removed RV2: 1Meg_log, 1.Custom footprints:Alpha_16mm_potentiometer
- removed RV3: 1Meg_lin, 1.Custom footprints:Alpha_16mm_potentiometer
- removed RV4: 100k_log, 1.Custom footprints:Alpha_16mm_potentiometer
- removed RV5: 10k_log, 1.Custom footprints:Alpha_16mm_potentiometer
- removed SW1: SPST, 1.Custom footprints:PinSocket_2x01_P2.54mm_Vertical_Wide
- added J10: Conn_01x01, Connector_PinSocket_2.54mm:PinSocket_1x01_P2.54mm_Vertical, F.Cu at (99.1, 68.6)
- added J11: Conn_01x01, Connector_PinSocket_2.54mm:PinSocket_1x01_P2.54mm_Vertical, F.Cu at (99.1, 94.0)
- added J12: Conn_01x01, Connector_PinSocket_2.54mm:PinSocket_1x01_P2.54mm_Vertical, F.Cu at (99.1, 109.2)
- added J5: Conn_01x01, Connector_PinSocket_2.54mm:PinSocket_1x01_P2.54mm_Vertical, F.Cu at (99.1, 48.3)
- added J7: Conn_01x01, Connector_PinSocket_2.54mm:PinSocket_1x01_P2.54mm_Vertical, F.Cu at (99.1, 43.2)
- added J8: Conn_01x01, Connector_PinSocket_2.54mm:PinSocket_1x01_P2.54mm_Vertical, F.Cu at (99.1, 81.3)
- added J9: Conn_01x01, Connector_PinSocket_2.54mm:PinSocket_1x01_P2.54mm_Vertical, F.Cu at (99.1, 86.4)
- D5: footprint 2.Breadboard components:D_Axial_Vertical -> 2.Breadboard components:D_Axial_Horizontal
- R1, R12, R2: footprint 2.Breadboard components:R_Axial_Horizontal -> 2.Breadboard components:R_Axial_Vertical
- moved J4 116.9 mm to (99.1, 35.6)
- moved C1 112.0 mm to (83.8, 27.9), turned to 270 degrees
- moved C3 104.7 mm to (58.4, 55.9), turned to 270 degrees
- moved R4 99.4 mm to (83.8, 53.3), turned to 180 degrees
- moved U2 97.1 mm to (61.0, 63.5), turned to 90 degrees
- moved C4 95.1 mm to (78.7, 58.4), turned to 270 degrees
- moved J2 95.1 mm to (99.1, 104.1)
- moved C9 94.3 mm to (66.0, 73.7)
- moved C8 94.3 mm to (73.7, 73.7)
- moved R10 94.3 mm to (73.7, 68.6)
- moved C12 92.7 mm to (78.7, 27.9), turned to 270 degrees
- moved J1 89.8 mm to (99.1, 73.7)
- moved U3 89.5 mm to (73.7, 96.5), turned to 90 degrees
- moved R17 87.4 mm to (78.7, 73.7), turned to 270 degrees
- moved R2 84.3 mm to (101.6, 76.2), turned to 270 degrees
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Connections:
- J2 pad 1: GND -> +4V5
- R7 pad 2: Net-(C5-Pad2) -> Net-(C5-Pad1)
Routing:
- net GND: track 0.00 -> 170.2 mm, vias 0 -> 13
- net +4V5: track 0.00 -> 83.8 mm, vias 0 -> 4
- net +9V: track 0.00 -> 45.7 mm, vias 0 -> 3
- net Net-(C8-Pad1): track 0.00 -> 38.1 mm, vias 0 -> 4
- net Net-(C5-Pad1): track 0.00 -> 35.6 mm, vias 0 -> 3
- net Net-(C5-Pad2): track 0.00 -> 30.5 mm, vias 0 -> 3
- net Net-(C2-Pad1): track 0.00 -> 20.3 mm
- net Net-(R17-Pad2): track 0.00 -> 20.3 mm, vias 0 -> 2
- net Net-(C2-Pad2): track 0.00 -> 17.8 mm, vias 0 -> 3
- net Net-(R4-Pad1): track 0.00 -> 15.2 mm, vias 0 -> 1
- net Net-(C7-Pad1): track 0.00 -> 12.7 mm, vias 0 -> 3
- net Net-(J11-Pad1): track 0.00 -> 12.7 mm
- net Net-(C11-Pad2): track 0.00 -> 10.2 mm, vias 0 -> 2
- net Net-(J9-Pad1): track 0.00 -> 10.2 mm, vias 0 -> 1
- net Net-(C11-Pad1): track 0.00 -> 10.2 mm, vias 0 -> 2
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Other:
- board outline added: 68.6 x 91.4 mm

Commit message: Finnished?
Parts:
- R1, R2, R8: footprint 2.Breadboard components:R_Axial_Vertical -> 2.Breadboard components:R_Axial_Horizontal
- moved R15 46.8 mm to (43.2, 66.0), turned to 90 degrees
- moved R16 37.5 mm to (48.3, 66.0)
- moved R13 35.4 mm to (50.8, 58.4)
- moved R14 34.2 mm to (45.7, 66.0), turned to 90 degrees
- moved R9 31.0 mm to (55.9, 33.0), turned to 180 degrees
- moved R7 30.7 mm to (63.5, 96.5)
- moved R19 29.0 mm to (66.0, 81.3)
- moved R18 29.0 mm to (50.8, 94.0)
- moved U3 28.4 mm to (45.7, 91.4)
- moved D3 28.1 mm to (68.6, 76.2), turned to 270 degrees
- moved R11 28.1 mm to (55.9, 99.1), turned to 0 degrees
- moved R12 27.9 mm to (55.9, 81.3)
- moved R8 27.0 mm to (53.3, 35.6), turned to 180 degrees
- moved C9 26.2 mm to (53.3, 50.8), turned to 0 degrees
- moved R2 25.5 mm to (76.2, 73.7), turned to 180 degrees
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Routing:
- net +9V: track 45.7 -> 148.2 mm, vias 3 -> 9
- net GND: track 170.2 -> 216.0 mm, vias 13 -> 15
- net +4V5: track 83.8 -> 119.4 mm
- net Net-(R15-Pad1): track 5.08 -> 27.9 mm
- net Net-(Q2-Pad1): track 5.08 -> 20.3 mm
- net Net-(D4-Pad2): track 7.62 -> 22.9 mm, vias 2 -> 4
- net Net-(J11-Pad1): track 12.7 -> 25.4 mm
- net Net-(R14-Pad1): track 7.62 -> 17.8 mm
- net Net-(C5-Pad1): track 35.6 -> 45.7 mm
- net Net-(D2-Pad2): track 0.00 -> 8.73 mm, vias 0 -> 2
- net Net-(C8-Pad1): track 38.1 -> 45.7 mm, vias 4 -> 2
- net Net-(Q2-Pad3): track 7.62 -> 15.2 mm
- net Net-(D5-Pad2): track 2.54 -> 10.2 mm
- net Net-(J9-Pad1): track 10.2 -> 17.8 mm
- net Net-(C9-Pad1): track 10.2 -> 15.2 mm
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Other:
- board size 68.6 x 91.4 mm -> 45.7 x 81.3 mm

Commit message: Its never done
Parts:
- removed RV1: 1Meg_lin, 1.Custom footprints:Alpha_16mm_potentiometer
- added J13: Conn_01x01, Connector_PinSocket_2.54mm:PinSocket_1x01_P2.54mm_Vertical, F.Cu at (78.7, 50.8)
- added J14: Conn_01x01, Connector_PinSocket_2.54mm:PinSocket_1x01_P2.54mm_Vertical, F.Cu at (78.7, 61.0)
- added J15: Conn_01x01, Connector_PinSocket_2.54mm:PinSocket_1x01_P2.54mm_Vertical, F.Cu at (78.7, 55.9)
- R3, R9: footprint 2.Breadboard components:R_Axial_Vertical -> 2.Breadboard components:R_Axial_Horizontal
- moved R9 10.2 mm to (45.7, 33.0), turned to 0 degrees
- moved D5 5.08 mm to (66.0, 43.2)
- moved R3 3.59 mm to (76.2, 33.0), turned to 180 degrees
- moved R4 2.54 mm to (73.7, 40.6)
- moved R6 2.54 mm to (66.0, 38.1)
- moved C11 2.54 mm to (71.1, 91.4)
- moved R17 2.54 mm to (55.9, 73.7)
Routing:
- net Net-(D4-Pad2): track 22.9 -> 17.8 mm, vias 4 -> 2
- net GND: track 216.0 -> 221.1 mm
- net Net-(J7-Pad1): track 5.08 -> 7.62 mm
- net Net-(J13-Pad1): track 17.8 -> 20.3 mm
- net Net-(D5-Pad2): track 10.2 -> 12.7 mm
- net Net-(R17-Pad2): track 25.4 -> 22.9 mm
- net Net-(C5-Pad2): track 33.0 -> 35.6 mm
- net Net-(C11-Pad2): track 10.2 -> 12.7 mm
- net Net-(C11-Pad1): track 12.7 -> 10.2 mm
Other:
- board size 45.7 x 81.3 mm -> 47 x 81.3 mm

Commit message: its never done
Parts:
- removed C12: 100n, 2.Breadboard components:C_Box_P5.08mm
- added D6: 1N4007, Diode_THT:D_DO-35_SOD27_P7.62mm_Horizontal, F.Cu at (109.2, 76.2)
- added D7: 1N4007, Diode_THT:D_DO-35_SOD27_P7.62mm_Horizontal, F.Cu at (109.2, 73.7)
- C1, C11, C7, C8, C9: footprint 2.Breadboard components:CP_Vertical -> Capacitor_THT:CP_Radial_D6.3mm_P2.50mm
- D1, D3: footprint 2.Breadboard components:LED_D3.0mm_Vertical -> LED_THT:LED_D3.0mm
- D2, D4: footprint 2.Breadboard components:D_Axial_Vertical -> Diode_THT:D_DO-35_SOD27_P7.62mm_Horizontal
- D5: footprint 2.Breadboard components:D_Axial_Horizontal -> Diode_THT:D_DO-35_SOD27_P7.62mm_Horizontal
- Q1: value Q_PMOS_GSD -> DMP3099L; moved to F.Cu
- R1, R10, R11, R13, R14, R15, R16, R17, R19, R2, R20, R3, R4, R5, R6, R7, R8, R9: footprint 2.Breadboard components:R_Axial_Horizontal -> Resistor_THT:R_Axial_DIN0204_L3.6mm_D1.6mm_P7.62mm_Horizontal
- R12, R18: footprint 2.Breadboard components:R_Axial_Vertical -> Resistor_THT:R_Axial_DIN0204_L3.6mm_D1.6mm_P7.62mm_Horizontal
- moved Q1 67.9 mm to (111.8, 85.1), turned to 180 degrees
- moved D2 65.1 mm to (109.2, 78.7), turned to 0 degrees
- moved C1 64.3 mm to (114.3, 67.3)
- moved J2 63.7 mm to (97.2, 43.2), turned to 180 degrees
- moved J3 60.8 mm to (105.4, 85.1), turned to 0 degrees
- moved R3 58.5 mm to (109.2, 81.3), turned to 0 degrees
- moved J12 57.8 mm to (93.3, 43.2), turned to 180 degrees
- moved C10 56.0 mm to (92.7, 46.4), turned to 270 degrees
- moved J4 52.8 mm to (97.2, 85.1), turned to 0 degrees
- moved R11 49.8 mm to (90.8, 63.5), turned to 90 degrees
- moved R18 46.0 mm to (80.0, 58.4)
- moved R5 45.2 mm to (106.7, 65.4), turned to 270 degrees
- moved C3 44.9 mm to (76.2, 68.6)
- moved R6 44.6 mm to (108.6, 51.4)
- moved D5 44.2 mm to (108.6, 55.2)
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Routing:
- net GND: track 221.1 -> 0.00 mm, vias 15 -> 0
- net +4V5: track 119.4 -> 64.3 mm, vias 4 -> 0
- net +9V: track 148.2 -> 107.5 mm, vias 9 -> 0
- net Net-(J15-Pad1): track 7.62 -> 45.6 mm
- net Net-(C8-Pad1): track 45.7 -> 16.3 mm, vias 2 -> 0
- net Net-(J5-Pad1): track 5.08 -> 31.5 mm, vias 1 -> 0
- net Net-(D6-Pad2): track 4.04 -> 28.7 mm
- net Net-(R15-Pad1): track 27.9 -> 5.08 mm, vias 1 -> 0
- net Net-(C2-Pad1): track 17.8 -> 34.5 mm
- net Net-(C11-Pad2): track 12.7 -> 27.2 mm, vias 2 -> 0
- net Net-(C9-Pad1): track 15.2 -> 29.0 mm, vias 2 -> 1
- net Net-(J13-Pad1): track 20.3 -> 8.43 mm, vias 1 -> 0
- net Net-(Q2-Pad1): track 20.3 -> 8.89 mm, vias 3 -> 0
- net Net-(R14-Pad1): track 17.8 -> 8.67 mm, vias 1 -> 0
- net Net-(C7-Pad1): track 10.2 -> 17.6 mm, vias 3 -> 0
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- added copper zone on B.Cu, net GND
- added copper zone on F.Cu, net GND
Other:
- board size 47 x 81.3 mm -> 61 x 52.1 mm
