File: engineers thumb.kicad_pcb (KiCad board)
At the start: 2 copper layers, 61 x 52.1 mm, 58 parts, among them J1 Conn_01x01, J10 Conn_01x01, J11 Conn_01x01, J12 Conn_01x01, J13 Conn_01x01, J14 Conn_01x01, J15 Conn_01x01, J2 Conn_01x01, J3 Conn_01x01, J4 Conn_01x01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

Commit message: Good progress made
Parts:
- removed J10, J11, J12, J13, J14, J15, J2, J3, J4, J5, J6, J7, J8, J9: Conn_01x01, Connector_PinSocket_2.54mm:PinSocket_1x01_P2.54mm_Vertical
- added RV1: 1Meg_lin, 1.Custom footprints:Alpha_16mm_potentiometer, B.Cu at (99.1, 55.9)
- added RV2: 1Meg_log, 1.Custom footprints:Alpha_16mm_potentiometer, B.Cu at (78.7, 55.9)
- added RV3: 1Meg_lin, 1.Custom footprints:Alpha_16mm_potentiometer, B.Cu at (58.4, 55.9)
- added RV4: 100k_log, 1.Custom footprints:Alpha_16mm_potentiometer, B.Cu at (58.4, 61.0)
- added RV5: 10k_log, 1.Custom footprints:Alpha_16mm_potentiometer, B.Cu at (99.1, 61.0)
- added SW1: SPST, 1.Custom footprints:PinSocket_2x01_P2.54mm_Vertical_Wide, B.Cu at (76.8, 95.9)
- J1: value Conn_01x01 -> Conn_01x04_Female; footprint Connector_PinSocket_2.54mm:PinSocket_1x01_P2.54mm_Vertical -> 1.Custom footprints:Molex_KK-254_01x04_P2.54mm_Right_Angle
- moved Q2 56.4 mm to (56.5, 96.5), turned to 90 degrees
- moved R16 54.6 mm to (59.7, 96.5), turned to 90 degrees
- moved U2 49.7 mm to (53.3, 85.1), turned to 90 degrees
- moved C10 48.6 mm to (76.2, 92.1), turned to 180 degrees
- moved C9 38.8 mm to (50.2, 88.9)
- moved R14 38.6 mm to (62.2, 88.9), turned to 270 degrees
- moved R15 38.1 mm to (64.8, 88.9), turned to 270 degrees
- moved R8 37.9 mm to (61.0, 74.9), turned to 180 degrees
- moved C7 37.6 mm to (61.0, 66.0)
- moved R10 37.5 mm to (50.8, 77.5), turned to 270 degrees
- moved R6 35.8 mm to (76.2, 66.7), turned to 90 degrees
- moved R5 35.6 mm to (71.1, 66.7), turned to 90 degrees
- moved R13 34.4 mm to (67.3, 88.9)
- moved C6 34.3 mm to (63.5, 80.0), turned to 270 degrees
- moved C8 32.6 mm to (53.3, 66.0)
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Connections:
- C11 pad 2: Net-(C11-Pad2) -> Output
- D6 pad 2: Net-(D6-Pad2) -> Vin
- J1 pad 1: Net-(J1-Pad1) -> Output
- Q1 pad 3: Net-(D6-Pad2) -> Vin
- R1 pad 1: Net-(J1-Pad1) -> Input
- R2 pad 1: Net-(J1-Pad1) -> Input
- R20 pad 2: Net-(C11-Pad2) -> Output
Routing:
- net Net-(C5-Pad2): track 30.0 -> 66.1 mm
- net Net-(D4-Pad1): track 10.6 -> 45.3 mm
- net Net-(RV1-Pad2): track 45.6 -> 16.1 mm
- net Net-(D6-Pad2): track 28.7 -> 0.00 mm
- net Net-(C11-Pad2): track 27.2 -> 0.00 mm
- net Net-(R5-Pad2): track 31.5 -> 8.94 mm
- net +4V5: track 64.3 -> 85.1 mm
- net Net-(C8-Pad1): track 16.3 -> 35.7 mm
- net Output: track 0.00 -> 19.3 mm
- net Vin: track 0.00 -> 18.9 mm
- net Net-(R6-Pad2): track 8.26 -> 25.8 mm
- net Net-(C9-Pad1): track 29.0 -> 15.3 mm, vias 1 -> 0
- net Net-(R14-Pad1): track 8.67 -> 21.7 mm
- net Net-(D4-Pad2): track 20.1 -> 10.2 mm
- net Net-(D2-Pad2): track 10.1 -> 19.7 mm
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- added copper zone on F.Cu, net +9V
- removed copper zone on F.Cu, net GND
Other:
- board size 61 x 52.1 mm -> 66 x 50.8 mm
- net class Default: clearance 0.508 -> 0.381
- rule trace_clearance: 0.508 -> 0.381
- board text added: "LM13700"
- board text added: "TL072"
