File: engineers thumb.sch (KiCad schematic (older format))
At the start: 58 parts, among them J1 Conn_01x01, J10 Conn_01x01, J11 Conn_01x01, J12 Conn_01x01, J13 Conn_01x01, J14 Conn_01x01, J15 Conn_01x01, J2 Conn_01x01, J3 Conn_01x01, J4 Conn_01x01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

Commit message: Good progress made
Parts:
- removed J1, J10, J11, J12, J13, J14, J15, J2, J3, J4, J5, J6, J7, J8, J9: Conn_01x01, Connector_PinSocket_2.54mm:PinSocket_1x01_P2.54mm_Vertical, symbol Connector:Conn_01x01_Female
- added J1: Conn_01x04_Female, 1.Custom footprints:Molex_KK-254_01x04_P2.54mm_Right_Angle, symbol Connector:Conn_01x04_Female
- added RV1, RV3: 1Meg_lin, 1.Custom footprints:Alpha_16mm_potentiometer, symbol Device:R_POT
- added RV2: 1Meg_log, 1.Custom footprints:Alpha_16mm_potentiometer, symbol Device:R_POT
- added RV4: 100k_log, 1.Custom footprints:Alpha_16mm_potentiometer, symbol Device:R_POT
- added RV5: 10k_log, 1.Custom footprints:Alpha_16mm_potentiometer, symbol Device:R_POT
- added SW1: SPST, 1.Custom footprints:PinSocket_2x01_P2.54mm_Vertical_Wide, symbol Switch:SW_SPST
Connections:
- net +4V5: now also RV5.1, SW1.2 (B)
- net GND: now also J1.3 (Pin_3)
- net at U3.7: now also RV5.2
- net Input: now reaches R1.1, R2.1
- net Input: now also J1.4 (Pin_4)
- net at C2.1, U1.3 (+): now also RV1.1
- net at C5.2, R17.1, U1.1: now also RV2.2, RV2.3, RV5.3
- net Output: now reaches C11.2, R20.2
- net Output: now also J1.1 (Pin_1)
- net Vin: now reaches D6.2 (A), Q1.3 (D)
- net Vin: now also J1.2 (Pin_2)
- net at R6.2: now also RV4.1
- net at R5.2: now also RV3.1
- net at C8.1, R10.1: now also RV3.2, RV3.3, RV4.2, RV4.3
- net at C10.1: now also SW1.1 (A)
- net at R4.1: now also RV1.3
- net at U1.5 (+): now also RV1.2
- net at R7.1: now also RV2.1
